File: PCB/Stadion_rychlomer.kicad_pcb (KiCad board)
At the start: 4 copper layers, 44 x 44 mm, 56 parts, among them J2 OLED I2C, J3 ICSP, J4 Conn_01x03_Pin, J5 SPÍD & PWR, J6 AUX DDAA, J7 ENG RPM, Q1 140817143200, Q2 PC817, U1 Mikroprofesor, U3 LM1117MP-5.0, Y1 16MHz

Commit message: Updated PNs, minor tweaks on PCB
Parts:
- D9: value SMCJ85CA -> PTVS8V5S1UTR-QX; footprint Diode_SMD:D_SOD-123F -> AERO_Diode_SMD:D_SOD-123FL
- FB5, FB6: value FerriteBead_Small -> FerriteBead_4A_180Ω
- turned D9 to 180 degrees
Connections:
- C5 pad 1: Net-(D9-A2) -> Net-(D9-K)
- D9 pad 1: GND -> Net-(D9-K)
- D9 pad 2: Net-(D9-A2) -> GND
- FB5 pad 2: Net-(D9-A2) -> Net-(D9-K)
- U3 pad 3: Net-(D9-A2) -> Net-(D9-K)
Routing:
- net Net-(D9-K): track 0.00 -> 12.0 mm
- net Net-(D9-A2): track 12.0 -> 0.00 mm
- net Net-(D2-A): track 15.5 -> 16.7 mm
- net +5V: track 118.4 -> 117.4 mm
- net GND: vias 92 -> 102
Other:
- board text added: "VIN 5V SPD GND"
- board text removed: "GND VIN 5V SPD GND"
