File: PCB/Stadion_rychlomer.kicad_sch (KiCad schematic)
At the start: 65 parts, among them J1 USB_B_Micro, J2 OLED I2C, J3 ICSP, J4 Conn_01x03_Pin, J5 SPÍD & PWR, J6 AUX DDAA, J7 ENG RPM, Q1 140817143200, Q2 PC817, U1 Mikroprofesor, U2 FT232RL, U3 LM1117MP-5.0, Y1 16MHz

Commit message: SCL SDA Fixed, minor edits
Connections:
- net I2C_SCL: now also U1.28 (PC5); no longer U1.27 (PC4)
- net I2C_SDA: now also U1.27 (PC4); no longer U1.28 (PC5)
Changed lines of the file:
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@@
 		)
 	)
-	(label "I2C_SDA"
+	(label "I2C_SCL"
 		(at 71.12 85.09 0)
 		(effects
@@
 		)
 	)
-	(label "I2C_SCL"
+	(label "I2C_SDA"
 		(at 71.12 82.55 0)
 		(effects

Commit message: Upravy Routingu
Other:
- note added: "https://cz.mouser.com/cs/c/semiconductors/power-management-ics/voltage-regulators-voltage-controllers/ldo-voltage-regulators/?input%20voltage%2C%20max=18%20V~~60%20V&number%20of%20outputs=1%20Output&output%20voltage=5%20V&package%20%2F%20case=SOT-89~~SOT-89-4%7C~SOT223-3%7C~SOT89-3&instock=y&rp=semiconductors%2Fpower-management-ics%2Fvoltage-regulators-voltage-controllers%2Fldo-voltage-regulators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"
- note added: "https://www.ti.com/lit/ds/symlink/tlv709.pdf?ts=1792494302204"
Changed lines of the file:
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@@
+		)
+	)
+	(text "https://cz.mouser.com/cs/c/semiconductors/power-management-ics/voltage-regulators-voltage-controllers/ldo-voltage-regulators/?input%20voltage%2C%20max=18%20V~~60%20V&number%20of%20outputs=1%20Output&output%20voltage=5%20V&package%20%2F%20case=SOT-89~~SOT-89-4%7C~SOT223-3%7C~SOT89-3&instock=y&rp=semiconductors%2Fpower-management-ics%2Fvoltage-regulators-voltage-controllers%2Fldo-voltage-regulators%7C~Package%20%2F%20Case%7C~Input%20Voltage%2C%20Max"
+		(exclude_from_sim no)
+		(at 220.726 5.08 0)
+		(effects
+			(font
+				(size 1.27 1.27)
+			)
 		)
 	)
@@
 		(effects
 			(font
+				(size 1.27 1.27)
+			)
+		)
+	)
+	(text "https://www.ti.com/lit/ds/symlink/tlv709.pdf?ts=1792494302204"
+		(exclude_from_sim no)
+		(at 219.964 15.494 0)
+		(effects
+			(font
