File: PCB_Speedo_UniFace/UniFace/UniFace.kicad_pcb (KiCad board)
At the start: 2 copper layers, 44 x 44 mm, 0 parts

Commit message: UniFace PCB
Routing:
- added copper zone on B.Cu, net GND
- added copper zone on F.Cu, net GND

Commit message: dalsi verze uniface
Other:
- outline, holes or cut-outs redrawn
