File: PCB_Stadi_Speedo_V2/Stadi_Speedo_V2.kicad_pcb (KiCad board)
At the start: 4 copper layers, 41.7 x 44 mm, 71 parts, among them J2 OLED I2C, J3 ICSP, J4 OLED SH1106, J5 SPÍD & PWR, J6 AUX DDAA, J7 ENG RPM, Q1 140817143200, Q2 PC817, U1 Mikroprofesor, U3 LM1117MP-5.0, U4 ME6211C33M5, Y1 16MHz

Commit message: update pcb V2
Parts:
- moved C23 4.35 mm to (120.4, 137.4), turned to 90 degrees
- moved C13 4.32 mm to (128.0, 137.5), turned to 90 degrees
- moved C12 4.30 mm to (125.5, 137.5), turned to 90 degrees
- moved C21 4.30 mm to (122.9, 137.4), turned to 90 degrees
- moved C20 2.91 mm to (122.9, 140.5), turned to 90 degrees
- moved C22 2.87 mm to (120.4, 140.5), turned to 90 degrees
- moved C18 2.84 mm to (125.5, 140.5), turned to 90 degrees
- moved C17 2.81 mm to (128.0, 140.5), turned to 90 degrees
- moved FB6 0.59 mm to (118.6, 156.8), turned to 0 degrees
- moved C2 0.24 mm to (122.4, 146.6)
- moved J4 0.24 mm to (126.7, 144.0)
- moved C3 0.19 mm to (122.1, 144.8)
Connections:
- C26 pad 2: VCC -> /OLED VCC
- C27 pad 2: VCC -> /OLED VCC
- J4 pad 28: VCC -> /OLED VCC
Routing:
- net +5V: track 66.2 -> 83.6 mm
- net /I2C_SCL: track 8.06 -> 24.9 mm
- net /I2C_SDA: track 9.65 -> 25.8 mm
- net /A0: track 27.8 -> 22.7 mm
- net /D5: track 27.6 -> 32.6 mm, vias 2 -> 1
- net VCC: track 8.75 -> 4.04 mm
- net /OLED VCC: track 0.00 -> 4.59 mm
- net /D13/SCK_: track 34.1 -> 37.4 mm
- net /D4: track 26.9 -> 25.0 mm, vias 2 -> 1
- net /A1: track 23.7 -> 22.1 mm
- net Net-(J5-Pin_4): track 5.23 -> 6.21 mm
- net /D11/MOSI_: track 21.8 -> 22.4 mm
Other:
- board text added: "A C D B"
- board text added: "ADDR"
- board text added: "IREF BRI"
- board text added: "MISO +5V"
- board text added: "RES"
- board text added: "RES GND"
- board text added: "SCK MOSI"
- board text added: "X27"
- board text added: "_"
- board text removed: "+5V MISO"
- board text removed: "GND 5V"
- board text removed: "GND RES"
- board text removed: "MOSI SCK"

Commit message: PCB V2 Update
Parts:
- removed the ? at (90.3, 150.0)
- removed the ? at (94.1, 131.0)
- added ?: , , F.Cu at (108.9, 154.3)
- added ?: , , F.Cu at (107.8, 136.5)
- added ?: , , F.Cu at (111.1, 152.9)
- added ?: , , F.Cu at (110.7, 136.5)
- added R19: 10K, Resistor_SMD:R_0603_1608Metric, B.Cu at (107.8, 139.0)
- added R21: 20K, Resistor_SMD:R_0603_1608Metric, B.Cu at (109.3, 139.0)
- added R22: 20K, Resistor_SMD:R_0603_1608Metric, B.Cu at (112.2, 139.0)
- added R23: 10K, Resistor_SMD:R_0603_1608Metric, B.Cu at (109.6, 150.4)
- added R23: 10K, Resistor_SMD:R_0603_1608Metric, B.Cu at (110.7, 139.0)
- added U5: MAX31855KASA, Package_SO:SOIC-8_3.9x4.9mm_P1.27mm, B.Cu at (110.0, 145.6)
- moved ? 16.8 mm to (103.1, 150.1), turned to 90 degrees
- moved ? 14.3 mm to (101.9, 136.7), turned to 90 degrees
- moved ? 12.6 mm to (105.6, 150.2)
- moved J3 0.46 mm to (102.4, 143.2)
- moved C6 0.12 mm to (122.9, 125.6)
- renumbered Q1 to OPT0, Q2 to OPTO
Connections:
- ? pad 2: (no net) -> VCC
- J4 pad 30: unconnected-(J4-Pin_30-Pad30) -> GND
- U1 pad 10: unconnected-(U1-PD6-Pad10) -> /D6/CS K
- U1 pad 11: unconnected-(U1-PD7-Pad11) -> /D7/SCK K
- U1 pad 12: unconnected-(U1-PB0-Pad12) -> /D8/SO K
Routing:
- net +3V3: track 22.0 -> 49.9 mm, vias 0 -> 2
- net /D6/CS K: track 0.00 -> 20.1 mm, vias 0 -> 2
- net /D7/SCK K: track 0.00 -> 19.6 mm, vias 0 -> 2
- net /D8/SO K: track 0.00 -> 17.1 mm, vias 0 -> 2
- net /RESET_: track 19.3 -> 28.6 mm
- net /T+: track 0.00 -> 7.11 mm
- net Net-(U5-~{CS}): track 0.00 -> 5.31 mm
- net /T-: track 0.00 -> 5.01 mm
- net Net-(U5-SCK): track 0.00 -> 4.87 mm
- net GND: track 13.7 -> 16.9 mm, vias 89 -> 108
- net +5V: track 83.6 -> 86.7 mm, vias 10 -> 8
- net /D5: track 32.6 -> 30.1 mm
- net Net-(D8-A2): track 23.1 -> 22.3 mm
- net /D13/SCK_: track 37.4 -> 38.0 mm
- net /D12/MISO_: track 27.0 -> 27.6 mm
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Other:
- board text added: "-BROD"
- board text added: "0.91 OLED"
- board text added: "31855"
- board text added: "ADR."
- board text added: "BRIGHT"
- board text added: "CHVOJKOVICE"
- board text added: "D4 D5 A1 A0"
- board text added: "D6"
- board text added: "D7"
- board text added: "G 5 S D"
- board text added: "IREF"
- board text added: "JESVS"
- board text added: "K TYPE"
- board text added: "KATODA"
- board text added: "LM1117"
- board text added: "MOPED JESVS"
- board text added: "MOSI"
- board text added: "MoPED"
- board text added: "OLOMóC"
- board text added: "PD2"
- board text added: "PD3"
- board text added: "PULLUPZZZ"
- board text added: "Q1"
- board text added: "Q2"
- board text added: "RPM GND"
- board text added: "SCK"
- board text added: "SENSE"
- board text added: "STADI SPíDO"
- board text added: "STEPPER"
- board text added: "STS"
- board text added: "T- T+"
- board text added: "TRMOCUPLE"
- board text added: "TVS"
- board text added: "V2"
- board text removed: "ADDR"
- board text removed: "AUX DDAA"
- board text removed: "IREF BRI"
- board text removed: "MOPeD JeSUS STADi-SPÍDo V2"
- board text removed: "SCK MOSI"
- board text removed: "STS CHVOJKOVICE-BROD / KATODA OLOMÓC"

Commit message: PCB Stadi Uniface
Parts:
- added ?: , , F.Cu at (125.6, 125.4)
- moved C6 0.58 mm to (122.4, 125.5)
- moved ? 0.54 mm to (106.0, 149.8), turned to 90 degrees
Routing:
- net +5V: track 86.7 -> 89.1 mm
- net GND: track 16.9 -> 19.2 mm, vias 108 -> 113
- net /D5: track 30.1 -> 30.8 mm
- net VCC: track 4.04 -> 3.40 mm
- net +3V3: track 49.9 -> 49.3 mm
Other:
- board text added: "NTC/"
- board text added: "STEPPER/"
- board text added: "STPR"
- board text removed: "STEPPER"

Commit message: drobné opravy tras + přidán schématický symbol čůráka
Routing:
- net /RESET_: track 28.6 -> 19.5 mm, vias 2 -> 1
- net +3V3: track 49.3 -> 40.8 mm
- net +5V: track 89.1 -> 81.7 mm, vias 8 -> 10
- net /D6/CS K: track 20.1 -> 17.2 mm
- net GND: vias 113 -> 119
Other:
- board text added: "A"
- board text added: "B"
- board text added: "C"
- board text added: "D"
- board text added: "G"
- board text added: "U"
- board text added: "o"
- board text removed: "A C D B"
